File: hardware/PGTN_daisy3_exp_32io.brd (EAGLE design)
At the start: 77.5 x 105.4 mm, 103 parts, among them IC6 MCP23S17SP, IC9 MCP23S17SP, Q1 2N3904, Q2 2N3904, Q3 2N3904, Q4 2N3904, Q5 2N3904, Q6 2N3904, Q7 2N3904, Q8 2N3904

Commit message: rename AnalogPin to AnalogInputPin
Parts:
- added BTN10, BTN11, BTN12, BTN13, BTN14, BTN15, BTN16, BTN9, GTIN10, GTIN11, GTIN12, GTIN13, GTIN14, GTIN15, GTIN16, GTIN9, LED1, LED10, LED11, LED12, LED13, LED14, LED15, LED16, LED2, LED3, LED4, LED5, LED6, LED7, LED8, LED9: HEADER/MALE/01, connectors:HEADER/MALE/01
- added Q10, Q11, Q12, Q13, Q14, Q15, Q16, Q9: 2N3904, transistors:TO92
- added R49, R53, R57, R61, R65, R69, R73, R77, R81, R82, R83: 1k, resistors:RESISTOR/7.5
- added R50, R54, R58, R62, R66, R70, R74, R78: 100k, resistors:RESISTOR/7.5
- added R51, R55, R59, R63, R67, R71, R75, R79: 1M, resistors:RESISTOR/7.5
- added R52, R56, R60, R64, R68, R72, R76, R80: 10k, resistors:RESISTOR/7.5
- moved BTN6 265.4 mm to (3.81, 82.5)
- moved BTN5 264.8 mm to (3.81, 85.1)
- moved BTN7 263.0 mm to (3.81, 80.0)
- moved BTN8 260.8 mm to (3.81, 77.5)
- moved GTIN5 259.2 mm to (1.27, 85.1)
- moved GTIN7 259.1 mm to (1.27, 80.0)
- moved GTIN6 257.2 mm to (1.27, 82.5)
- moved GTIN8 256.7 mm to (1.27, 77.5)
- moved R48 236.1 mm to (26.7, 59.7)
- moved R36 231.0 mm to (26.7, 74.9)
- moved R40 230.2 mm to (26.7, 69.8)
- moved R42 230.0 mm to (11.4, 64.8)
- moved R44 229.9 mm to (26.7, 64.8)
- moved R46 229.9 mm to (11.4, 59.7)
- moved R45 228.5 mm to (26.7, 57.1)
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Connections:
- removed net 29: 29.1
- removed net 30: 30.1
- removed net N$23: 14_RX.1
- removed net N$28: 13_TX.1
- removed net N$42: 7_CS.1
- removed net N$47: 6_SD_CLK.1
- removed net N$53: 5_SD_CMD.1
- removed net N$61: 4_SD_D0.1
- removed net N$62: 3_SD_D1.1
- removed net N$63: 2_SD_D2.1
- removed net N$64: 1_SD_D3.1
- removed net N$65: 0.1
- removed net N$73: 5V.1
- removed net VDD: IC6.9, IC9.9
- removed net VSS: IC6.10, IC9.10
- new net 25_GTIN1: IC9.23, R57.2
- new net 25_GTIN10: IC9.26, R69.2
- new net 25_GTIN11: IC9.27, R73.2
- new net 25_GTIN12: IC9.28, R77.2
- new net 25_GTIN2: IC9.24, R61.2
- new net 25_GTIN9: IC9.25, R65.2
- new net N$100: LED16.1, R8.2
- new net N$101: IC6.18, R81.2
- new net N$102: IC9.18, R82.2
- new net N$108: IC9.15, R83.2
- new net N$34: 8_SCK.1, IC6.12, IC9.12
- new net N$35: 10_MOSI.1, IC6.13, IC9.13
- new net N$36: 11.1, IC6.11
- new net N$38: BTN9.1, GTIN9.1, R50.1
- new net N$40: Q9.1, R49.1, R52.1
- new net N$41: BTN10.1, GTIN10.1, R54.1
- new net N$43: Q10.2, R54.2, R55.2
- new net N$44: Q10.1, R53.1, R56.1
- new net N$45: BTN11.1, GTIN11.1, R58.1
- new net N$46: Q11.2, R58.2, R59.2
- new net N$48: Q11.1, R57.1, R60.1
- new net N$49: BTN12.1, GTIN12.1, R62.1
- new net N$50: Q12.2, R62.2, R63.2
- new net N$51: Q12.1, R61.1, R64.1
- new net N$52: BTN13.1, GTIN13.1, R66.1
- new net N$74: BTN14.1, GTIN14.1, R70.1
- new net N$75: Q14.2, R70.2, R71.2
- new net N$76: Q14.1, R69.1, R72.1
- new net N$77: BTN15.1, GTIN15.1, R74.1
- new net N$78: Q15.2, R74.2, R75.2
- new net N$79: Q15.1, R73.1, R76.1
- new net N$80: BTN16.1, GTIN16.1, R78.1
- new net N$81: Q16.2, R78.2, R79.2
- new net N$82: Q16.1, R77.1, R80.1
- new net N$83: IC9.21, R49.2
- new net N$84: IC9.22, R53.2
- new net N$85: LED1.1, R9.2
- new net N$86: LED2.1, R10.2
- new net N$87: LED3.1, R11.2
- new net N$88: LED4.1, R12.2
- new net N$89: LED5.1, R13.2
- new net N$90: LED6.1, R14.2
- new net N$91: LED7.1, R15.2
- new net N$92: LED8.1, R16.2
- new net N$93: LED9.1, R1.2
- new net N$94: LED10.1, R2.2
- new net N$95: LED11.1, R3.2
- new net N$96: LED12.1, R4.2
- new net N$97: LED13.1, R5.2
- new net N$98: LED14.1, R6.2
- new net N$99: LED15.1, R7.2
- net +5V: now also IC6.9, IC9.9, R52.2, R56.2, R60.2, R64.2, R68.2, R72.2, R76.2, R80.2, R81.1, R82.1, R83.1
- net N$33: now also 9_MISO.1, IC6.14, IC9.14; no longer 10_MOSI.1
- net N$37: now also 12.1, IC9.11; no longer 9_MISO.1
- net N$39: now also Q9.2, R50.2, R51.2; no longer 8_SCK.1
- net N$66: now also Q13.2, R66.2, R67.2; no longer 11.1
- net N$67: now also Q13.1, R65.1, R68.1; no longer 12.1
- net PE: now also IC6.10, IC6.15, IC6.16, IC6.17, IC9.10, IC9.16, IC9.17, Q10.3, Q11.3, Q12.3, Q13.3, Q14.3, Q15.3, Q16.3, Q9.3, R51.1, R55.1, R59.1, R63.1, R67.1, R71.1, R75.1, R79.1
Routing:
- net +5V: track 0.00 -> 191.9 mm
- net N$34: track 0.00 -> 149.6 mm, vias 0 -> 1
- net N$33: track 0.00 -> 71.8 mm
- net N$35: track 0.00 -> 71.4 mm, vias 0 -> 2
- net N$37: track 0.00 -> 70.9 mm, vias 0 -> 1
- net 25_GTIN6: track 0.00 -> 52.2 mm
- net N$92: track 0.00 -> 48.7 mm, vias 0 -> 1
- net N$94: track 0.00 -> 48.7 mm
- net N$91: track 0.00 -> 48.7 mm
- net N$93: track 0.00 -> 47.7 mm, vias 0 -> 1
- net N$90: track 0.00 -> 46.1 mm
- net N$36: track 0.00 -> 41.9 mm, vias 0 -> 1
- net N$95: track 0.00 -> 39.5 mm
- net N$96: track 0.00 -> 36.9 mm
- net N$89: track 0.00 -> 36.9 mm
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Other:
- board size 77.5 x 105.4 mm -> 78.8 x 105.4 mm
- board text added: "1"
- board text added: "10"
- board text added: "11"
- board text added: "12"
- board text added: "13"
- board text added: "14"
- board text added: "15"
- board text added: "16"
- board text added: "2"
- board text added: "3"
- board text added: "4"
- board text added: "5"
- board text added: "6"
- board text added: "7"
- board text added: "8"
- board text added: "9"
- board text added: "OUTPUTS"
