File: hardware/PGTN_daisy3_exp_32io.sch (EAGLE design)
At the start: 97 parts, among them IC6 MCP23S17SP, IC9 MCP23S17SP, Q1 2N3904, Q2 2N3904, Q3 2N3904, Q4 2N3904, Q5 2N3904, Q6 2N3904, Q7 2N3904, Q8 2N3904

Commit message: rename AnalogPin to AnalogInputPin
Parts:
- added BTN10, BTN11, BTN12, BTN13, BTN14, BTN15, BTN16, BTN9, GTIN10, GTIN11, GTIN12, GTIN13, GTIN14, GTIN15, GTIN16, GTIN9, LED1, LED10, LED11, LED12, LED13, LED14, LED15, LED16, LED2, LED3, LED4, LED5, LED6, LED7, LED8, LED9: HEADER/MALE/01, connectors:HEADER/MALE/01
- added Q10, Q11, Q12, Q13, Q14, Q15, Q16, Q9: 2N3904, transistors:2N3904
- added R49, R53, R57, R61, R65, R69, R73, R77, R81, R82, R83: 1k, resistors:RESISTORRESISTOR/UPRIGHT/7.5
- added R50, R54, R58, R62, R66, R70, R74, R78: 100k, resistors:RESISTORRESISTOR/UPRIGHT/7.5
- added R51, R55, R59, R63, R67, R71, R75, R79: 1M, resistors:RESISTORRESISTOR/UPRIGHT/7.5
- added R52, R56, R60, R64, R68, R72, R76, R80: 10k, resistors:RESISTORRESISTOR/UPRIGHT/7.5
Connections:
- removed net 29: 29.3
- removed net 30: 30.3
- removed net N$23: 14_RX.3
- removed net N$28: 13_TX.3
- removed net N$42: 7_CS.3
- removed net N$47: 6_SD_CLK.3
- removed net N$53: 5_SD_CMD.3
- removed net N$61: 4_SD_D0.3
- removed net N$62: 3_SD_D1.3
- removed net N$63: 2_SD_D2.3
- removed net N$64: 1_SD_D3.3
- removed net N$65: 0.3
- removed net N$73: 5V.3
- new net 25_GTIN1: IC9.GPA2, R57.2
- new net 25_GTIN10: IC9.GPA5, R69.2
- new net 25_GTIN11: IC9.GPA6, R73.2
- new net 25_GTIN12: IC9.GPA7, R77.2
- new net 25_GTIN2: IC9.GPA3, R61.2
- new net 25_GTIN9: IC9.GPA4, R65.2
- new net N$100: LED16.3, R8.2
- new net N$101: IC6.!RESET, R81.2
- new net N$102: IC9.!RESET, R82.2
- new net N$108: IC9.A0, R83.2
- new net N$34: 8_SCK.3, IC6.SCK, IC9.SCK
- new net N$35: 10_MOSI.3, IC6.SI, IC9.SI
- new net N$36: 11.3, IC6.!CS
- new net N$38: BTN9.3, GTIN9.3, R50.1
- new net N$40: Q9.C, R49.1, R52.1
- new net N$41: BTN10.3, GTIN10.3, R54.1
- new net N$43: Q10.B, R54.2, R55.2
- new net N$44: Q10.C, R53.1, R56.1
- new net N$45: BTN11.3, GTIN11.3, R58.1
- new net N$46: Q11.B, R58.2, R59.2
- new net N$48: Q11.C, R57.1, R60.1
- new net N$49: BTN12.3, GTIN12.3, R62.1
- new net N$50: Q12.B, R62.2, R63.2
- new net N$51: Q12.C, R61.1, R64.1
- new net N$52: BTN13.3, GTIN13.3, R66.1
- new net N$74: BTN14.3, GTIN14.3, R70.1
- new net N$75: Q14.B, R70.2, R71.2
- new net N$76: Q14.C, R69.1, R72.1
- new net N$77: BTN15.3, GTIN15.3, R74.1
- new net N$78: Q15.B, R74.2, R75.2
- new net N$79: Q15.C, R73.1, R76.1
- new net N$80: BTN16.3, GTIN16.3, R78.1
- new net N$81: Q16.B, R78.2, R79.2
- new net N$82: Q16.C, R77.1, R80.1
- new net N$83: IC9.GPA0, R49.2
- new net N$84: IC9.GPA1, R53.2
- new net N$85: LED1.3, R9.2
- new net N$86: LED2.3, R10.2
- new net N$87: LED3.3, R11.2
- new net N$88: LED4.3, R12.2
- new net N$89: LED5.3, R13.2
- new net N$90: LED6.3, R14.2
- new net N$91: LED7.3, R15.2
- new net N$92: LED8.3, R16.2
- new net N$93: LED9.3, R1.2
- new net N$94: LED10.3, R2.2
- new net N$95: LED11.3, R3.2
- new net N$96: LED12.3, R4.2
- new net N$97: LED13.3, R5.2
- new net N$98: LED14.3, R6.2
- new net N$99: LED15.3, R7.2
- net +5V: now also IC6.VDD, IC9.VDD, R52.2, R56.2, R60.2, R64.2, R68.2, R72.2, R76.2, R80.2, R81.1, R82.1, R83.1
- net N$33: now also 9_MISO.3, IC6.SO, IC9.SO; no longer 10_MOSI.3
- net N$37: now also 12.3, IC9.!CS; no longer 9_MISO.3
- net N$39: now also Q9.B, R50.2, R51.2; no longer 8_SCK.3
- net N$66: now also Q13.B, R66.2, R67.2; no longer 11.3
- net N$67: now also Q13.C, R65.1, R68.1; no longer 12.3
- net PE: now also IC6.A0, IC6.A1, IC6.A2, IC6.VSS, IC9.A1, IC9.A2, IC9.VSS, Q10.E, Q11.E, Q12.E, Q13.E, Q14.E, Q15.E, Q16.E, Q9.E, R51.1, R55.1, R59.1, R63.1, R67.1, R71.1, R75.1, R79.1
Other:
- note added: "INPUTS"
- note added: "OUTPUTS"
- moved on the sheet: 0, 10_MOSI, 11, 12, 13_TX, 14_RX, 1_SD_D3, 2_SD_D2, 3.3V, 3.3V1, 3_SD_D1, 4_SD_D0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
